Commit message: Update treewheel_mobile.urdf

File: urdf/treewheel_mobile.urdf (robot description, URDF)
Before this commit: robot treewheel_mobile, 5 links, 4 joints
Links:
- added link top_structure, mass 0.0001; collision box size=0.09 0.09 0.01; visual box size=0.151 0.0999 0.03
- link base_link: mass 0.10052 -> 0.12; geometry collision mesh filename=package://mobile_robot/meshes/base_link.STL; visual mesh filename=package://mobile_robot/meshes/base_link.STL
- link castor: mass 0.042129 -> 0.046; geometry collision mesh filename=package://mobile_robot/meshes/castor.STL; visual mesh filename=package://mobile_robot/meshes/castor.STL
- link castor_wheel: mass 0.0082874 -> 0.0088; geometry collision mesh filename=package://mobile_robot/meshes/castor_wheel.STL; visual mesh filename=package://mobile_robot/meshes/castor_wheel.STL
- link left_wheel: mass 0.021404 -> 0.14; geometry collision mesh filename=package://mobile_robot/meshes/left_wheel.STL; visual mesh filename=package://mobile_robot/meshes/left_wheel.STL
- link right_wheel: geometry collision mesh filename=package://mobile_robot/meshes/right_wheel.STL; visual mesh filename=package://mobile_robot/meshes/right_wheel.STL
Joints:
- added joint structure_joint: type fixed, parent base_link, child top_structure, origin xyz=0 0 0.005 rpy=0 0 0
- joint castorjoint: limit effort=10 velocity=10 -> (none); origin xyz=0.072581 0 -0.0025 rpy=0 0 0 -> xyz=0.072581 0 -0.0025 rpy=0 0 -3.142
- joint castorwheel: limit effort=10 velocity=10 -> (none); origin xyz=0.015014 0.00014167 -0.02296 rpy=-1.5708 0 0 -> xyz=-0.015 0 -0.023 rpy=1.5708 0 0
- joint leftwheel: limit effort=10 velocity=10 -> (none)
- joint rightwheel: limit effort=10 velocity=10 -> (none)
